File: hardware/sg75.kicad_sch (KiCad schematic)
At the start: 165 parts

Commit message: begin pcb design
Parts:
- removed D1, D10, D11, D12, D13, D14, D15, D16, D17, D18, D19, D2, D20, D21, D22, D23, D24, D25, D26, D27, D28, D29, D3, D30, D31, D32, D33, D34, D35, D36, D37, D38, D39, D4, D40, D41, D42, D43, D44, D45, D46, D47, D48, D49, D5, D50, D51, D52, D53, D54, D55, D56, D57, D58, D59, D6, D60, D61, D62, D63, D64, D65, D66, D67, D68, D69, D7, D70, D71, D72, D73, D74, D75, D76, D77, D78, D79, D8, D80, D81, D82, D9: D_Small, symbol Device:D_Small
- removed MX1, MX10, MX11, MX12, MX13, MX14, MX15, MX16, MX17, MX18, MX19, MX2, MX20, MX21, MX22, MX23, MX24, MX25, MX26, MX27, MX28, MX29, MX3, MX30, MX31, MX32, MX33, MX34, MX35, MX36, MX37, MX38, MX39, MX4, MX40, MX41, MX42, MX43, MX44, MX45, MX46, MX47, MX48, MX49, MX5, MX50, MX51, MX52, MX53, MX54, MX55, MX56, MX57, MX58, MX59, MX6, MX60, MX61, MX62, MX63, MX64, MX65, MX66, MX67, MX68, MX69, MX7, MX70, MX71, MX72, MX73, MX74, MX75, MX76, MX77, MX78, MX79, MX8, MX80, MX81, MX82, MX9: ~, symbol Keyboard:MX_Switch
- removed S1: PEC11R-4215F-S0024, digikey-footprints:Rotary_Encoder_Switched_PEC11R, symbol dk_Encoders:PEC11R-4215F-S0024
Other:
- added sheet MCU (MCU.kicad_sch)
- added sheet key-matrix (key-matrix.kicad_sch)
- note added: "${CURRENT_DATE}"
- note added: "sg75 Key Matrix"
- note added: "v1.0"
- note removed: "'""
- note removed: ",<"
- note removed: "-_"
- note removed: ".>"
- note removed: "/?"
- note removed: "0)"
- note removed: "1!"
- note removed: "2@"
- note removed: "3#"
- note removed: "4$"
- note removed: "5%"
- note removed: "6^"
- note removed: "7&"
- note removed: "8*"
- note removed: "9("
- note removed: ";:"
- note removed: "=+"
- note removed: "A"
- note removed: "B"
- note removed: "BKSP"
- note removed: "C"
- note removed: "CAPS"
- note removed: "D"
- note removed: "DEL"
- note removed: "DOWN"
- note removed: "E"
- note removed: "ENTER"
- note removed: "ESC"
- note removed: "F"
- note removed: "F1"
- note removed: "F10"
- note removed: "F11"
- note removed: "F12"
- note removed: "F2"
- note removed: "F3"
- note removed: "F4"
- note removed: "F5"
- note removed: "F6"
- note removed: "F7"
- note removed: "F8"
- note removed: "F9"
- note removed: "FN"
- note removed: "G"
- note removed: "H"
- note removed: "I"
- note removed: "INS"
- note removed: "J"
- note removed: "K"
- note removed: "L"
- note removed: "LALT"
- note removed: "LCTRL"
- note removed: "LEFT"
- note removed: "LSHIFT"
- note removed: "M"
- note removed: "N"
- note removed: "O"
- note removed: "P"
- note removed: "PG DN"
- note removed: "PG UP"
- note removed: "PRTSC"
- note removed: "Q"
- note removed: "R"
- note removed: "RALT"
- note removed: "RCTRL"
- note removed: "RIGHT"
- note removed: "ROTARY ENCODER"
- note removed: "RSHIFT"
- note removed: "S"
- note removed: "SPACE"
- note removed: "T"
- note removed: "TAB"
- note removed: "U"
- note removed: "UP"
- note removed: "V"
- note removed: "W"
- note removed: "WIN"
- note removed: "X"
- note removed: "Y"
- note removed: "Z"
- note removed: "[{"
- note removed: "\|"
- note removed: "]}"
- note removed: "`~"
