File: hardware/MCU.kicad_sch (KiCad schematic)
At the start: 16 parts, among them J1 781710004, SW1 SW_Push, U1 ATmega32U4-A, Y1 16MHz

Commit message: finish pcb
Parts:
- removed F1: 500mA, Fuse:Fuse_1206_3216Metric, symbol Device:Polyfuse
- C7: footprint Diode_SMD:D_SOD-123 -> Capacitor_SMD:C_0805_2012Metric
Connections:
- net VCC is gone; now on net +5V: J1.1
- net ROW2: now reaches U1.1 (PE6)
- net ROW1: now reaches U1.10 (PB2)
- net COL9: now reaches U1.11 (PB3)
- net COL10: now reaches U1.18 (PD0)
- net COL11: now reaches U1.19 (PD1)
- net COL12: now reaches U1.20 (PD2)
- net COL13: now reaches U1.21 (PD3)
- net COL14: now reaches U1.22 (PD5)
- net COL15: now reaches U1.25 (PD4)
- net ENC_UP: now reaches U1.26 (PD6)
- net ENC_DOWN: now reaches U1.27 (PD7)
- net ROW6: now reaches U1.28 (PB4)
- net COL4: now reaches U1.29 (PB5)
- net D-: now reaches R3.2, U1.3 (D-)
- net COL5: now reaches U1.30 (PB6)
- net COL1: now reaches U1.32 (PC7)
- net COL2: now reaches U1.36 (PF7)
- net COL3: now reaches U1.37 (PF6)
- net COL6: now reaches U1.38 (PF5)
- net ROW3: now reaches U1.39 (PF4)
- net D+: now reaches R2.2, U1.4 (D+)
- net ROW5: now reaches U1.40 (PF1)
- net COL7: now reaches U1.41 (PF0)
- net ROW4: now reaches U1.8 (PB0)
- net COL8: now reaches U1.9 (PB1)
- no-connect marks 2 -> 3
