File: hardware/key-matrix.kicad_sch (KiCad schematic)
At the start: 165 parts

Commit message: finish pcb
Parts:
- added D83: D_Small, Diode_SMD:D_SOD-123, symbol Device:D_Small
Connections:
- net COL10: now also MX50.1; no longer MX56.1
- net COL11: now also MX56.1; no longer MX62.1
- net COL12: now also MX62.1; no longer MX68.1
- net COL13: now also MX68.1; no longer MX73.1, MX74.1
- net COL14: now also MX73.1, MX74.1; no longer MX78.1
- net COL15: now also MX78.1
- net COL9: no longer MX50.1
- net ROW1: now also D83.1 (K); no longer S1.1
- net GND: now reaches S1.3
- net GND: now also S1.C (COM)
- net ENC_UP: now reaches S1.A (CH_A)
- net ENC_DOWN: now reaches S1.B (CH_B)
- new net: D83.2 (A), S1.1
Other:
- moved on the sheet: S1
