File: hardware/sg75.kicad_pcb (KiCad board)
At the start: 2 copper layers, 181 parts, among them J1 781710004, SW1 SW_Push, U1 ATmega32U4-A, Y1 16MHz

Commit message: finish pcb
Parts:
- removed F1: 500mA, Fuse:Fuse_1206_3216Metric
- added D83: D_Small, Diode_SMD:D_SOD-123, B.Cu at (629.4, 31.8)
- moved R2 359.8 mm to (489.7, 122.2)
- moved R3 358.2 mm to (489.7, 124.6)
- moved J1 347.3 mm to (481.1, 127.5), turned to 0 degrees
- moved C5 326.2 mm to (499.0, 122.9), turned to 90 degrees
- moved C3 326.1 mm to (502.2, 141.1)
- moved C2 324.8 mm to (506.2, 125.2), turned to 90 degrees
- moved R4 323.8 mm to (508.6, 125.2)
- moved R1 323.8 mm to (491.1, 141.0)
- moved C6 323.8 mm to (508.4, 136.2)
- moved C7 323.8 mm to (508.6, 129.9)
- moved U1 323.8 mm to (496.6, 133.0)
- moved Y1 323.8 mm to (508.6, 133.0)
- moved C1 323.7 mm to (496.6, 123.7), turned to 90 degrees
- moved SW1 323.7 mm to (516.5, 130.7)
- moved C4 321.8 mm to (486.7, 130.2), turned to 180 degrees
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Connections:
- net Net-(U1-D+) renamed D+
- net Net-(U1-D-) renamed D-
- J1 pad 1: VCC -> +5V
- MX50 pad 1: COL9 -> COL10
- MX56 pad 1: COL10 -> COL11
- MX62 pad 1: COL11 -> COL12
- MX68 pad 1: COL12 -> COL13
- MX73 pad 1: COL13 -> COL14
- MX74 pad 1: COL13 -> COL14
- MX78 pad 1: COL14 -> COL15
- S1 pad 1: ROW1 -> Net-(D83-A)
- S1 pad 3: unconnected-(S1-Pad3) -> GND
- S1 pad A: unconnected-(S1-CH_A-PadA) -> ENC_UP
- S1 pad B: unconnected-(S1-CH_B-PadB) -> ENC_DOWN
- S1 pad C: unconnected-(S1-COM-PadC) -> GND
- U1 pad 1: unconnected-(U1-PE6-Pad1) -> ROW2
- U1 pad 10: unconnected-(U1-PB2-Pad10) -> ROW1
- U1 pad 11: unconnected-(U1-PB3-Pad11) -> COL9
- U1 pad 18: unconnected-(U1-PD0-Pad18) -> COL10
- U1 pad 19: unconnected-(U1-PD1-Pad19) -> COL11
- U1 pad 20: unconnected-(U1-PD2-Pad20) -> COL12
- U1 pad 21: unconnected-(U1-PD3-Pad21) -> COL13
- U1 pad 22: unconnected-(U1-PD5-Pad22) -> COL14
- U1 pad 25: unconnected-(U1-PD4-Pad25) -> COL15
- U1 pad 26: unconnected-(U1-PD6-Pad26) -> ENC_UP
- U1 pad 27: unconnected-(U1-PD7-Pad27) -> ENC_DOWN
- U1 pad 28: unconnected-(U1-PB4-Pad28) -> ROW6
- U1 pad 29: unconnected-(U1-PB5-Pad29) -> COL4
- U1 pad 30: unconnected-(U1-PB6-Pad30) -> COL5
- U1 pad 32: unconnected-(U1-PC7-Pad32) -> COL1
- U1 pad 36: unconnected-(U1-PF7-Pad36) -> COL2
- U1 pad 37: unconnected-(U1-PF6-Pad37) -> COL3
- U1 pad 38: unconnected-(U1-PF5-Pad38) -> COL6
- U1 pad 39: unconnected-(U1-PF4-Pad39) -> ROW3
- U1 pad 40: unconnected-(U1-PF1-Pad40) -> ROW5
- U1 pad 41: unconnected-(U1-PF0-Pad41) -> COL7
- U1 pad 8: unconnected-(U1-PB0-Pad8) -> ROW4
- U1 pad 9: unconnected-(U1-PB1-Pad9) -> COL8
Routing:
- net ROW1: track 0.00 -> 408.5 mm, vias 0 -> 2
- net ROW6: track 0.00 -> 399.1 mm, vias 0 -> 2
- net ROW2: track 0.00 -> 385.1 mm, vias 0 -> 2
- net ROW3: track 0.00 -> 379.4 mm, vias 0 -> 2
- net ROW4: track 0.00 -> 334.5 mm, vias 0 -> 2
- net ROW5: track 0.00 -> 324.9 mm, vias 0 -> 2
- net COL15: track 0.00 -> 265.5 mm, vias 0 -> 1
- net COL1: track 0.00 -> 265.5 mm, vias 0 -> 1
- net ENC_DOWN: track 0.00 -> 256.0 mm
- net ENC_UP: track 0.00 -> 249.8 mm, vias 0 -> 1
- net COL2: track 0.00 -> 248.2 mm, vias 0 -> 1
- net COL14: track 0.00 -> 243.0 mm, vias 0 -> 1
- net COL13: track 0.00 -> 231.5 mm, vias 0 -> 1
- net COL12: track 0.00 -> 217.2 mm, vias 0 -> 1
- net COL3: track 0.00 -> 216.0 mm, vias 0 -> 1
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- added copper zone on B.Cu, net GND
- added copper zone on F.Cu, net GND
Other:
- board outline added: 314.3 x 123.8 mm
- board text removed: "update molex footprint"
